File: schematics/submarineCard.kicad_sch (KiCad schematic)
At the start: 21 parts, among them M1 Motor_DC, Q4 NMOS, U2 3MP SPI Camera, U4 MPU-6050

Commit message: schematic
added temp sensor, startet work on new motor circut, changes to handcontroller
Parts:
- removed D6: D, symbol Device:D
- added T2: ~, Sensor_Audio:Infineon_PG-LLGA-5-2, symbol Sensor_Audio:IM73A135V01
- R3: value 5K -> 2.6
- renumbered WS1 to T1
Connections:
- net +5V: now also T2.2 (V_{CC})
- net Earth: now also T2.3 (GND), T2.4 (GND)
- net at A3.A10: now also T2.1 (OUT)
- net at A3.A11: now also T1.1 (OUT)
- net at A3.A4: no longer T1.1 (OUT)
- net at D5.1 (K): no longer M1.1 (+)
- net -12V: no longer names the net of M1.2 (-)
- net P2A0 renamed P3A0
- net P2A1 renamed P3A1
- net P2A3 renamed P3A2
- net P3A2: no longer A3.D12
- new net P3A3: A3.D12
Other:
- moved on the sheet: T1

Commit message: added motorCard
Parts:
- removed C3: 10mF, symbol Device:C
- removed D5: D, symbol Device:D
- removed LD1: ~, symbol Device:D_Laser_1A3C
- removed M1: Motor_DC, symbol Motor:Motor_DC
- removed Q4: NMOS, symbol Simulation_SPICE:NMOS
- removed R3: 2.6, symbol Device:R
- removed R5: 112, symbol Device:R
- renumbered R4 to R1, R6 to R2, R7 to R3, R8 to R4
Connections:
- net P5A1: now reaches A3.D4
- net P3GND: now reaches A3.GND1 (GND)
- net P5A2: now reaches A3.GND2 (GND)
Other:
- moved on the sheet: LD1

Commit message: new motor
Parts:
- added C1: 047uF, symbol Device:C
- added M3: Motor_DC, symbol Motor:Motor_DC
- added R10: 10k, symbol Device:R
- added R11: 14K, symbol Device:R
- added R9: 33K, symbol Device:R
- added U1: OPA1622, Package_SON:Texas_S-PVSON-N10, symbol Amplifier_Audio:OPA1622
Connections:
- net Earth: now also C1.2, M3.2 (-), R10.2
- net P5A1: no longer names the net of A3.D4
- net P5A1: now also R9.1
- new net: R10.1, R11.1, U1.10 (-)
- new net: M3.1 (+), R11.2, U1.9
- new net: C1.1, R9.2, U1.1 (+)
Other:
- moved on the sheet: M1, M2
